File: encoder-board.kicad_pcb (KiCad board)
At the start: 2 copper layers, 101.6 x 39.4 mm, 21 parts, among them J1 PMOD, SW1 Bourns PEC11R-4220F-S0024, SW2 Bourns PEC11R-4220F-S0024, SW3 Bourns PEC11R-4220F-S0024, SW4 Bourns PEC11R-4220F-S0024, SW5 Sparkfun-Button, SW6 Sparkfun-Button, SW7 Sparkfun-Button, SW8 Sparkfun-Button, U1 74LS165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

Commit message: Added a label to the silkscreen
Parts:
- moved H3 5.74 mm to (166.4, 106.7)
Routing:
- net /DOUT: track 111.2 -> 112.3 mm
Other:
- board text added: "4x Encoder +4x Button Rev.1"
- board text added: "PMOD"
Changed lines of the file:
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@@
   (general
     (thickness 1.6)
-    (drawings 4)
+    (drawings 6)
     (tracks 245)
     (zones 0)
@@
   )
   (module MountingHole:MountingHole_2.5mm (layer F.Cu)
-    (at 160.655 106.172)
+    (at 166.37 106.68)
     (descr "Mounting Hole 2.5mm, no annular")
     (tags "mounting hole 2.5mm no annular")
@@
       (rotate (xyz 0 0 0))
     )
+  )
+  (gr_text "   4x Encoder\n+4x Button\nRev.1" (at 156.21 107.315) (layer F.SilkS)
+    (effects (font (size 1.5 1.5) (thickness 0.3)))
+  )
+  (gr_text PMOD (at 107.95 105.41 90) (layer F.SilkS)
+    (effects (font (size 1.5 1.5) (thickness 0.3)))
   )
   (gr_line (start 102.87 85.09) (end 102.87 124.46) (layer Edge.Cuts) (width 0.15))
@@
   (segment (start 188.976 105.156) (end 188.976 110.236) (width 0.25) (layer B.Cu) (net 19))
   (segment (start 188.976 110.236) (end 177.8 121.412) (width 0.25) (layer B.Cu) (net 19))
-  (via (at 107.95 110.49) (size 0.8) (drill 0.4) (layers F.Cu B.Cu) (net 19))
+  (via (at 109.855 104.14) (size 0.8) (drill 0.4) (layers F.Cu B.Cu) (net 19))
+  (segment (start 105.156 104.14) (end 109.855 104.14) (width 0.25) (layer F.Cu) (net 19))
+  (segment (start 109.855 111.055685) (end 109.855 110.49) (width 0.25) (layer F.Cu) (net 19))
+  (segment (start 109.855 104.14) (end 109.855 104.705685) (width 0.25) (layer B.Cu) (net 19))
+  (segment (start 111.252 121.412) (end 109.855 120.015) (width 0.25) (layer F.Cu) (net 19))
   (segment (start 156.464006 121.412) (end 111.252 121.412) (width 0.25) (layer F.Cu) (net 19))
-  (segment (start 111.252 121.412) (end 107.95 118.11) (width 0.25) (layer F.Cu) (net 19))
-  (segment (start 107.95 111.055685) (end 107.95 110.49) (width 0.25) (layer F.Cu) (net 19))
-  (segment (start 107.95 118.11) (end 107.95 111.055685) (width 0.25) (layer F.Cu) (net 19))
-  (via (at 107.950006 104.14) (size 0.8) (drill 0.4) (layers F.Cu B.Cu) (net 19))
-  (segment (start 105.156 104.14) (end 107.950006 104.14) (width 0.25) (layer F.Cu) (net 19))
-  (segment (start 107.95 104.140006) (end 107.950006 104.14) (width 0.25) (layer B.Cu) (net 19))
-  (segment (start 107.95 110.49) (end 107.95 104.140006) (width 0.25) (layer B.Cu) (net 19))
+  (via (at 109.855 110.49) (size 0.8) (drill 0.4) (layers F.Cu B.Cu) (net 19))
+  (segment (start 109.855 120.015) (end 109.855 111.055685) (width 0.25) (layer F.Cu) (net 19))
+  (segment (start 109.855 104.705685) (end 109.855 110.49) (width 0.25) (layer B.Cu) (net 19))
   (segment (start 200.56 114.34) (end 188.06 114.34) (width 0.25) (layer F.Cu) (net 21))
   (segment (start 188.06 114.34) (end 186.504366 114.34) (width 0.25) (layer F.Cu) (net 21))
